File: Wiring/PCB.kicad_pcb (KiCad board)
At the start: 2 copper layers, 80.7 x 114.3 mm, 18 parts, among them J1 Conn_01x04_Pin, J2 Conn_01x08_Pin, SW1 SW_Push, SW2 SW_Push, U1 DHT11, U2 XIAO-ESP32-C3-SMD

Commit message: kk
Parts:
- moved G*** 2.24 mm to (135.0, 119.5)
Changed lines of the file:
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@@
 	(footprint "LOGO"
 		(layer "F.Cu")
-		(at 137 120.5)
+		(at 135 119.5)
 		(property "Reference" "G***"
 			(at 0 0 0)
